Commit message: fwd_kin

File: urdf/scara_modified.urdf.xacro (robot description, xacro)
@@ -111,5 +111,5 @@
     <visual>
       <geometry>
-        <cylinder radius="0.05" length="0.8"/>
+        <cylinder radius="0.05" length="0.8"/> <!--EE starts at -0.4 Z wrt J3-->
       </geometry>
       <origin xyz="0 0 0"/>

Commit message: Part 1 and 2-a

File: urdf/scara_modified.urdf.xacro (robot description, xacro)
@@ -26,5 +26,5 @@
     </inertial>
   </link>
-  <joint name="joint1" type="revolute"> <!-- Joint 1 that connects base to link1 -->
+  <joint name="joint1" type="fixed"> <!-- was revolute-->
     <parent link="base_link"/>
     <child link="link1"/>
@@ -60,5 +60,5 @@
   </link>
   <!-- Joint 2 -->
-  <joint name="joint2" type="revolute">
+  <joint name="joint2" type="fixed">  <!-- was revolute-->
     <parent link="link1"/>
     <child link="link2"/>
@@ -155,4 +155,5 @@
       <state_interface name="position"/>
       <state_interface name="velocity"/>
+      <state_interface name="effort"/>    <!-- added this so effort would show number instead of nan -->
     </joint>
   </ros2_control>

Commit message: assignment 2

File: urdf/scara_modified.urdf.xacro (robot description, xacro)
@@ -10,17 +10,17 @@
     <visual>
       <geometry>
-        <cylinder radius="0.1" length="1.5"/>
+        <cylinder radius="0.5" length="7.5"/>
       </geometry>
-      <origin xyz="0 0 0.75"/>
+      <origin xyz="0 0 3.75"/>
     </visual>
     <collision>
       <geometry>
-        <cylinder radius="0.1" length="1.5"/>
+        <cylinder radius="0.5" length="7.5"/>
       </geometry>
-      <origin xyz="0 0 0.75"/>
+      <origin xyz="0 0 3.75"/>
     </collision>
     <inertial>
-      <mass value="1.0"/>
-      <inertia ixx="0.01" iyy="0.01" izz="0.01"
+      <mass value="20.0"/>
+      <inertia ixx="30" iyy="30" izz="30"
                ixy="0" ixz="0" iyz="0"/> <!--using some junk values so that gazebo doens't cause issues -->
     </inertial>
@@ -29,5 +29,5 @@
     <parent link="base_link"/>
     <child link="link1"/>
-    <origin xyz="0 0 1.5"/> <!--definig link1 at 1.5m from the  base about z-->
+    <origin xyz="0 0 7.5"/> <!--definig link1 at 1.5m from the  base about z-->
     <axis xyz="0 0 1"/>     <!--defining j1 axis of rotatoin along z axis-->
     <limit lower="-3.14" upper="3.14" effort="100" velocity="1.0"/> <!-- making sure the joint goes from -pi to pi. dummy values for effort and velocity-->
@@ -37,5 +37,5 @@
     <visual>
         <geometry>    <!-- adding a joint cylinder that makes it look connected. It is only visual-->
-            <cylinder radius="0.12" length="0.12"/>
+            <cylinder radius="0.6" length="0.6"/>
         </geometry>
         <origin xyz="0 0 0"/>
@@ -43,17 +43,17 @@
     <visual><!--Actual link display -->
       <geometry>
-        <cylinder radius="0.05" length="0.8"/>
+        <cylinder radius="0.25" length="4.0"/>
       </geometry>
-      <origin xyz="0.4 0 0" rpy="0 1.5708 0"/> <!--rotating it to make it horizontal-->
+      <origin xyz="2 0 0" rpy="0 1.5708 0"/> <!--rotating it to make it horizontal-->
     </visual>
     <collision>
       <geometry>
-        <cylinder radius="0.05" length="0.8"/>
+        <cylinder radius="0.25" length="4.0"/>
       </geometry>
-      <origin xyz="0.4 0 0" rpy="0 1.5708 0"/>
+      <origin xyz="2 0 0" rpy="0 1.5708 0"/>
     </collision>
     <inertial>
-      <mass value="1.0"/>
-      <inertia ixx="0.01" iyy="0.01" izz="0.01"
+      <mass value="10"/>
+      <inertia ixx="30" iyy="30" izz="30"
                ixy="0" ixz="0" iyz="0"/>
     </inertial>
@@ -63,5 +63,5 @@
     <parent link="link1"/>
     <child link="link2"/>
-    <origin xyz="0.8 0 0.1"/> <!--0.1 vertical offeset to match the diagram-->
+    <origin xyz="4 0 0.5"/> <!--0.1 vertical offeset to match the diagram-->
     <axis xyz="0 0 1"/> <!--J2 axis along z axis-->
     <limit lower="-3.14" upper="3.14" effort="100" velocity="1.0"/>
@@ -71,29 +71,29 @@
     <visual>
         <geometry>    <!-- adding a joint cylinder that makes it look connected. It is only visual-->
-            <cylinder radius="0.12" length="0.24"/>
+            <cylinder radius="0.6" length="1.2"/>
         </geometry>
-        <origin xyz="0 0 -0.12"/>
+        <origin xyz="0 0 -0.6"/>
     </visual>
     <visual>  <!--housing for the prismatic jooint-->
       <geometry>
-        <box size="0.1 0.1 0.3"/>
+        <box size="0.5 0.5 1.5"/>
       </geometry>
-      <origin xyz="0.6 0 0"/> <!--offset to match J3-->
+      <origin xyz="3 0 0"/> <!--offset to match J3-->
     </visual>
     <visual><!--actual link display -->
       <geometry>
-        <cylinder radius="0.05" length="0.6"/>
+        <cylinder radius="0.25" length="3.0"/>
       </geometry>
-      <origin xyz="0.3 0 0" rpy="0 1.5708 0"/> <!--horizontal arm-->
+      <origin xyz="1.5 0 0" rpy="0 1.5708 0"/> <!--horizontal arm-->
     </visual>
     <collision>
       <geometry>
-        <cylinder radius="0.05" length="0.6"/>
+        <cylinder radius="0.25" length="3.0"/>
       </geometry>
-      <origin xyz="0.3 0 0" rpy="0 1.5708 0"/>
+      <origin xyz="1.5 0 0" rpy="0 1.5708 0"/>
     </collision>
     <inertial>
-      <mass value="1.0"/>
-      <inertia ixx="0.01" iyy="0.01" izz="0.01"
+      <mass value="10"/>
+      <inertia ixx="30" iyy="30" izz="30"
                ixy="0" ixz="0" iyz="0"/>
     </inertial>
@@ -103,7 +103,7 @@
     <parent link="link2"/>
     <child link="link3"/>
-    <origin xyz="0.6 0 0"/>
+    <origin xyz="3 0 0"/>
     <axis xyz="0 0 1"/><!--keeping the z axis aligned but negating range to match diagram and have tool come down-->
-    <limit lower="-0.5" upper="0" effort="100" velocity="1.0"/>
+    <limit lower="-2.5" upper="0" effort="100000" velocity="5.0"/>
   </joint>
   <!-- Link 3-->
@@ -111,5 +111,5 @@
     <visual>
       <geometry>
-        <cylinder radius="0.05" length="0.8"/> <!--EE starts at -0.4 Z wrt J3-->
+        <cylinder radius="0.25" length="4.0"/> <!--EE starts at -0.4 Z wrt J3-->
       </geometry>
       <origin xyz="0 0 0"/>
@@ -117,20 +117,20 @@
     <collision>
       <geometry>
-        <cylinder radius="0.05" length="0.8"/>
+        <cylinder radius="0.25" length="4.0"/>
       </geometry>
       <origin xyz="0 0 0"/>
     </collision>
     <inertial>
-      <mass value="0.5"/>
-      <inertia ixx="0.01" iyy="0.01" izz="0.01"
+      <mass value="10"/>
+      <inertia ixx="30" iyy="30" izz="30"
                ixy="0" ixz="0" iyz="0"/>
     </inertial>
   </link>
   <!-- ros2_control interface -->
-  <ros2_control name="scara_system" type="system">
+  <!-- <ros2_control name="scara_system" type="system">
     <hardware>
       <plugin>gazebo_ros2_control/GazeboSystem</plugin>
     </hardware>
-    <joint name="joint1">
+   <joint name="joint1">
       <command_interface name="position">
         <param name="min">-3.14</param>
@@ -150,18 +150,18 @@
     <joint name="joint3">
       <command_interface name="effort">
-        <param name="min">-0.5</param>
-        <param name="max">0.0</param>
+        <param name="min">-100000.0</param>
+        <param name="max">100000.0</param>
       </command_interface>
       <state_interface name="position"/>
       <state_interface name="velocity"/>
-      <state_interface name="effort"/>    <!-- added this so effort would show instead of nan -->
+      <state_interface name="effort"/>
     </joint>
-  </ros2_control>
+  </ros2_control>-->
   <!-- Gazebo ros2_control plugin -->
   <gazebo>
-    <plugin name="gazebo_ros2_control"
-            filename="libgazebo_ros2_control.so">
-      <parameters>/home/$(env USER)/ros2_ws/install/scara_robot/share/scara_robot/config/scara_controllers.yaml</parameters>
-    </plugin> <!--changing this to get environ variable for user -->
+    <plugin name="joint_state_publisher" filename="libgazebo_ros_joint_state_publisher.so">
+      <joint_name>joint3</joint_name>
+      <update_rate>100</update_rate>
+    </plugin>
   </gazebo>
 </robot>
